Commit message: Finishing the ball logic and starting the robot madification and control

File: exp_assignment2/urdf/robot.xacro (robot description, xacro)
@@ -117,13 +117,13 @@
   <link name="camera_link">
 	    <collision>
-	      <origin xyz="0 0 0.025" rpy="0 0 0"/>
+	      <origin xyz="0 0 0.25" rpy="0 0 0"/>
 	      <geometry>
-		<box size="0.05 0.05 0.05"/>
+		<box size="0.025 0.025 0.5"/>
 	      </geometry>
 	    </collision>
 	    <visual>
-	      <origin xyz="0 0 0.025" rpy="0 0 0"/>
+	      <origin xyz="0 0 0.25" rpy="0 0 0"/>
 	      <geometry>
-		<box size="0.05 0.05 0.05"/>
+		<box size="0.025 0.025 0.5"/>
 	      </geometry>
 	      <material name="red">
@@ -137,7 +137,8 @@
 	    </inertial>
   </link>
-  <joint name="camera_joint" type="fixed">
-	    <axis xyz="0 1 0" />
-	    <origin xyz="0.23 0 0.0" rpy="0 0 0"/>
+  <joint name="camera_joint" type="revolute">
+	    <axis xyz="0 0 1" />
+	    <origin xyz="0.0 0 0.035" rpy="0 0 0"/>
+	    <limit effort="1000.0" lower="-3.14" upper="3.14" velocity="0.2"/>
 	    <parent link="link_chassis"/>
 	    <child link="camera_link"/>

Commit message: Commitment
In this commitment I introduced the camera to the robot structure and added to it the ball tracking algorithm,
I modified the ball logic to comply to the play and normal behavior.
Finally I started working on the pet behaviors to keep track of the other modifications

File: exp_assignment2/urdf/robot.xacro (robot description, xacro)
@@ -115,15 +115,15 @@
     <joint_properties damping="1.0" friction="1.0"/>
   </joint>
-  <link name="camera_link">
+  <link name="neck_link">
 	    <collision>
 	      <origin xyz="0 0 0.25" rpy="0 0 0"/>
 	      <geometry>
-		<box size="0.025 0.025 0.5"/>
+		<box size="0.07 0.07 0.3"/>
 	      </geometry>
 	    </collision>
 	    <visual>
-	      <origin xyz="0 0 0.25" rpy="0 0 0"/>
+	      <origin xyz="0 0 0.15" rpy="0 0 0"/>
 	      <geometry>
-		<box size="0.025 0.025 0.5"/>
+		<box size="0.07 0.07 0.3"/>
 	      </geometry>
 	      <material name="red">
@@ -137,10 +137,48 @@
 	    </inertial>
   </link>
-  <joint name="camera_joint" type="revolute">
+  <joint name="neck_joint" type="revolute">
 	    <axis xyz="0 0 1" />
-	    <origin xyz="0.0 0 0.035" rpy="0 0 0"/>
-	    <limit effort="1000.0" lower="-3.14" upper="3.14" velocity="0.2"/>
+	    <limit effort="1000.0" lower="-1.8" upper="1.8" velocity="0.5"/>
+	    <origin xyz="0.15 0 0.035" rpy="0 0 0"/>
 	    <parent link="link_chassis"/>
+	    <child link="neck_link"/>
+	 </joint>
+  <link name="camera_link">
+	    <collision>
+	      <origin xyz="0 0 0.25" rpy="0 0 0"/>
+	      <geometry>
+		<box size="0.2 0.1 0.1"/>
+	      </geometry>
+	    </collision>
+	    <visual>
+	      <origin xyz="0 0 0.05" rpy="0 0 0"/>
+	      <geometry>
+		<box size="0.2 0.1 0.1"/>
+	      </geometry>
+	      <material name="red">
+		<color rgba="1 0 0 1"/>
+	      </material>
+	    </visual>
+	    <inertial>
+	      <mass value="1e-5" />
+	      <origin xyz="0 0 0" rpy="0 0 0"/>
+	      <inertia ixx="1e-6" ixy="0" ixz="0" iyy="1e-6" iyz="0" izz="1e-6" />
+	    </inertial>
+  </link>
+  <joint name="camera_joint" type="fixed">
+	    <axis xyz="1 0 0" />
+	    <origin xyz="0.025 0 0.30" rpy="0 0 0"/>
+	    <parent link="neck_link"/>
 	    <child link="camera_link"/>
 	 </joint>
+<transmission name="neck_joint_trans">
+	<type>transmission_interface/SimpleTransmission</type>
+	<joint name="neck_joint">
+		<hardwareInterface>hardware_interface/VelocityJointInterface</hardwareInterface>
+	</joint>
+	<actuator name="motor1">
+		<hardwareInterface>hardware_interface/VelocityJointInterface</hardwareInterface>
+		<mechanicalInterface>1</mechanicalInterface>
+	</actuator>
+</transmission>
 </robot>

Commit message: Finished functionalities
All functionalities are up and running, just one contingency is left that is when the ball is in the peripheral vision and close to the robot, it is really difficult for him to center it: the robot tend to go around the target

File: exp_assignment2/urdf/robot.xacro (robot description, xacro)
@@ -132,12 +132,11 @@
 	    </visual>
 	    <inertial>
-	      <mass value="1e-5" />
+	      <mass value="2" />
 	      <origin xyz="0 0 0" rpy="0 0 0"/>
-	      <inertia ixx="1e-6" ixy="0" ixz="0" iyy="1e-6" iyz="0" izz="1e-6" />
+	      <inertia ixx="1e-4" ixy="0" ixz="0" iyy="1e-4" iyz="0" izz="1e-5" />
 	    </inertial>
   </link>
-  <joint name="neck_joint" type="revolute">
+  <joint name="neck_joint" type="fixed">
 	    <axis xyz="0 0 1" />
-	    <limit effort="1000.0" lower="-1.8" upper="1.8" velocity="0.5"/>
 	    <origin xyz="0.15 0 0.035" rpy="0 0 0"/>
 	    <parent link="link_chassis"/>
@@ -166,13 +165,14 @@
 	    </inertial>
   </link>
-  <joint name="camera_joint" type="fixed">
-	    <axis xyz="1 0 0" />
+  <joint name="camera_joint" type="revolute">
+	    <axis xyz="0 0 1" />
+	    <limit effort="1000.0" lower="-1.8" upper="1.8" velocity="0.5"/>
 	    <origin xyz="0.025 0 0.30" rpy="0 0 0"/>
 	    <parent link="neck_link"/>
 	    <child link="camera_link"/>
 	 </joint>
-<transmission name="neck_joint_trans">
+<transmission name="camera_joint_trans">
 	<type>transmission_interface/SimpleTransmission</type>
-	<joint name="neck_joint">
+	<joint name="camera_joint">
 		<hardwareInterface>hardware_interface/VelocityJointInterface</hardwareInterface>
 	</joint>
